File: Hardware/eagle/calculator_15-Digit.sch (EAGLE design)
At the start: 141 parts, among them M1 IRLML2244, M10 IRLML2244, M11 IRLML2244, M3 IRLML2244, M4 IRLML2244, M5 IRLML2244, M6 IRLML2244, M7 IRLML2244, M8 IRLML2244, M9 IRLML2244, U1 74HC4051_MUX, U3 ATMEGA1284P-PU, U4 TLV70033, X1 MICROMATCH-12, X3 MICROMATCH-12, Y2 12MHz

Commit message: New Hardware Design V0.4a
Parts:
- removed C13: 15n, rcl:C-EU025_050-025X075
- removed D10, D9: SD103CW, BaseApp:DIODESMA
- removed S1: RESET, _jc:10-XX
- removed U$1: IRLML6244, transistor-power:IRLML2502
- removed X2, X4: (no value), pinhead:PINHD-2X6
- added C12: 0.1uF, SparkFun:CAP0805
- added C9: 1µ, rcl:C-EU025_050-025X075
- added D11, D12: SD103CW, BaseApp:DIODESMA
- added M2: IRLML2244, IRLML6402:IRLML6402
- added R27: 6k8, rcl:R-EU_R1206
- added R28, R44: 47k, rcl:R-EU_0204/7
- C18: value 15n -> 100n
- C4: value 2µ2 -> 1µ; device _jc:C-US025_050-025X075 -> rcl:C-EU025_050-025X075
- R1: value 68k -> 47k
- R26, R3: value 27k -> 6k8
- R31, R32: value 39 -> 100
Connections:
- net D8 renamed D2_
- net SCL renamed D16_
- net SDA renamed D17_
- removed net 3V3: C1.1, C16.1, C2.1, C20.+, C3.1, C6.1, D5.C, D6.C, D7.A, R1.1, R21.1, R22.1, R4.1, U3.VCC, U4.OUT
- removed net D10: JP13.9, U3.PB4, X2.7
- removed net D15: U3.PB1
- removed net D18: D10.A, U$1.G, U3.PC2
- removed net D19: JP14.7, U3.PC3, X4.7
- removed net D2: JP1.1, U3.PD2
- removed net D20: JP14.6, U3.PC4, X4.6
- removed net D21: JP14.5, U3.PC5, X4.5
- removed net D22: JP14.4, U3.PC6, X4.4
- removed net D23: JP14.3, U3.PC7, X4.3
- removed net D3: JP2.1, U3.PD3
- removed net D5: JP13.8, U3.PD5, X2.6
- removed net D6: JP13.7, U3.PD6, X2.5
- removed net D7: U3.PD7
- removed net D9: U3.PB3
- removed net IO: U$2.D, U1.IO
- removed net IO_A__: JP13.11, X2.9
- removed net IO_B__: JP13.12, X2.10
- removed net IO_C__: JP13.13, X2.11
- removed net IO_D__: JP13.14, X2.12
- removed net N$7: D8.C
- removed net XX4: C14.2, C15.2, R32.1, SG1.2
- new net CA_PWM1: D12.A, M2.D
- new net D10_: JP1.1, JP13.10, U3.PD2
- new net D11_: JP13.8, JP2.1, U3.PD3
- new net D13_: JP13.7, U3.PD5
- new net D14_: JP14.1, U3.PD6
- new net D15_: JP14.2, U3.PD7
- new net D18_: R44.2, U3.PC2
- new net D19_: JP14.3, U3.PC3
- new net D1_: JP13.14, U3.PB1
- new net D20_: JP14.4, U3.PC4
- new net D21_: JP14.5, U3.PC5
- new net D22_: JP14.6, U3.PC6
- new net D23_: JP14.7, U3.PC7
- new net D3_: JP13.11, U3.PB3
- new net D4_: U3.PB4
- new net EN_: D11.C, D12.C, R27.1
- new net GND-ISO: C1.2, C12.2, C14.2, C15.2, C2.2, C3.2, C4.2, C6.2, C7.2, C8.2, D4.C, D5.A, JP5.GND, JP6.1, JP6.2, U$2.D, U1.INH, U1.IO, U1.VEE, U1.VSS, U3.GND, U3.GND_2
- new net N$10: C15.1, C9.2, R32.1, SG1.2
- new net N$8: M2.G, R28.2, R44.1
- net /RESET: no longer S1.S, S1.S1
- net A0: no longer C15.1
- net A5: now also KP1.C2, KP2.C2; no longer KP1.C0, KP2.C0
- net A7: now also KP1.C0, KP2.C0; no longer KP1.C2, KP2.C2
- net AREF: now also C12.1; no longer C13.1
- net CA_PWM: no longer X4.8
- net D0_: now also JP13.13
- net D12_: no longer D9.A, D9.C, U$1.D, U$1.S
- net D5_: no longer JP13.10, X2.8
- net D6_: now also JP13.12; no longer JP14.1, X4.1
- net D7_: now also JP13.9; no longer JP14.2, X4.2
- net EN: now also R27.2; no longer D10.C
- net GND: no longer C1.2, C13.2, C2.2, C3.2, C4.2, C6.2, C7.2, C8.2, D4.C, D5.A, JP5.GND, JP6.1, JP6.2, S1.P, S1.P1, U1.INH, U1.VEE, U1.VSS, U3.GND, U3.GND_2
- net IO_A: no longer X2.4
- net IO_B: no longer X2.3
- net IO_C: no longer X2.2
- net IO_D: no longer X2.1
- net IO_DP: no longer X4.9
- net IO_E: no longer X4.12
- net IO_F: no longer X4.11
- net IO_G: no longer X4.10
- net N$23: now also C9.1
- net VCC: now also C1.1, C16.1, C2.1, C20.+, C3.1, C6.1, D5.C, D6.C, D7.A, D8.C, M2.S, R1.1, R21.1, R22.1, R28.1, R4.1, U3.VCC, U4.OUT
- net XX_3: now also D11.A
Other:
- moved on the sheet: C10, C14, C15, JP13, JP14, R26, R3, R31, R32, R48, Y2
