File: Hardware/eagle/calculator_15-Digit.sch (EAGLE design)
At the start: 142 parts, among them M1 IRLML2244, M10 IRLML2244, M11 IRLML2244, M2 IRLML2244, M3 IRLML2244, M4 IRLML2244, M5 IRLML2244, M6 IRLML2244, M7 IRLML2244, M8 IRLML2244, M9 IRLML2244, U1 74HC4051_MUX, U3 ATMEGA1284P-PU, U4 TLV70033, X1 MICROMATCH-12, X3 MICROMATCH-12, Y2 12MHz

Commit message: Display .. 5x LTD040AUE-101A 3-digit_Display
Parts:
- added D10, D9: SD103CW, BaseApp:DIODESMA
- added IC1: MCP170333MB, linear:MCP170333MB
- added M12: IRLML2244, IRLML6402:IRLML6402
- added R45: 56R, rcl:R-EU_R1206
- added R46, R47: 47k, rcl:R-EU_0204/7
- added U$1: BATTERY-CHARGER-LI-PROT, diy-modules:BATTERY-CHARGER-LI-PROT
- added U$3: HT7333, HT7333_SOT89:HT7333
- C5: value 15n -> 100n
Connections:
- new net B_MINUS: BH8.-, U$1.B-
- new net CA_PWM2: D11.A, M12.D
- new net N$13: R45.2, U$1.IN+
- new net N$9: M12.G, R46.2, R47.1
- new net P2: BH10.-, BH12.-
- new net P3: BH11.+, BH9.+
- new net VIN_P: D10.A, D9.A, R45.1, R47.2
- net GND: now also IC1.GND, U$1.IN-, U$1.OUT-, U$3.GND
- net NC1: no longer BH11.+, BH9.+
- net NC3: no longer BH10.-, BH12.-, BH8.-
- net VCC: now also IC1.VO, R50.2, U$3.VOUT
- net V_IN: now also D9.C, IC1.VI1, U$1.B+, U$1.OUT+
- net XX_3: now also D10.C, M12.S, R46.1; no longer D11.A
Other:
- note added: "HT7333-A"
