File: Hardware/eagle/snc98_main_cpu.brd (EAGLE design)
At the start: 168.2 x 30 mm, 89 parts, among them IC1 MCP170333MB, M1 IRLML2244, M12 IRLML2244, M2 IRLML2244, M3 IRLML2244, T1 BCR135, T2 BCR135, T3 BCR185, U1 74HC4051_MUX, U2 DS18B20, U3 ATMEGA1284P-PU, U4 TLV70033 / TC1185, Y2 12MHz

Commit message: V 5.0 Hardware - Design
Parts:
- removed JP5: ICSP, _jc:2X3_LOCK
- added JP1: ICSP, _jc:2X3_SMD_VERTICAL
- C12: value 47n -> 220n
- C2: value 100nF -> 220nF
- C20, C21: value 10uF -> 4.7uF
- C7, C8: value 22pF -> 15pF
- R25: value 1k -> 100
- moved BH9 0.51 mm to (108.3, 23.5)
- moved C3 0.51 mm to (109.9, 17.3)
- moved BH10 0.51 mm to (46.6, 23.5)
- moved M1 0.25 mm to (128.8, 3.94)
- moved BH12 0.25 mm to (58.3, 23.5)
- moved R33 0.25 mm to (44.1, 14.6)
- moved BH11 0.25 mm to (96.6, 23.5)
- moved R35 0.13 mm to (49.0, 13.3)
Connections:
- net /RESET: now also JP1.P$1; no longer JP5.2
- net D5_: now also JP1.3; no longer JP5.3
- net D6_: now also JP1.6; no longer JP5.6
- net D7_: now also JP1.4; no longer JP5.4
- net GND-ISO: now also JP1.1; no longer JP5.1
- net VCC: now also JP1.5; no longer JP5.5
Routing:
- net VCC: track 234.1 -> 253.5 mm, vias 13 -> 15
- net DTR: track 77.3 -> 82.1 mm
- net GND: track 179.6 -> 182.9 mm
- net D7_: track 78.9 -> 81.7 mm
- net V_IN: track 262.6 -> 263.9 mm
- net P2: track 18.5 -> 19.3 mm
- net P3: track 18.5 -> 19.3 mm
- net D6_: track 89.5 -> 90.2 mm
- net D5_: track 65.5 -> 66.3 mm
- net GND-ISO: track 328.9 -> 329.0 mm, vias 15 -> 18
Other:
- outline, holes or cut-outs redrawn
