File: Hardware/eagle/snc98_main_cpu.brd (EAGLE design)
At the start: 168.2 x 30 mm, 89 parts, among them IC1 MCP170333MB, M1 IRLML2244, M12 IRLML2244, M2 IRLML2244, M3 IRLML2244, M4 IRLML6244, T1 BCR135, T2 BCR135, T3 BCR185, U1 74HC4051_MUX, U2 DS18B20, U3 ATMEGA1284P-PU, U4 TLV70033 / TC1185, Y2 12MHz

Commit message: add factorial() - today from -72 to +72.
add factorial() - today from -72 to +72.
Parts:
- C3: value 1µ -> 4µ7
Routing:
- net VCC: track 858.7 -> 858.1 mm

Commit message: add_prozent
Parts:
- moved R22 0.46 mm to (56.4, 3.94)
- moved 44 0.36 mm to (58.7, 4.06)
- moved R21 0.28 mm to (54.1, 4.45)
- moved C22 0.25 mm to (50.0, 7.37)
Routing:
- net GND-ISO: track 1019.6 -> 925.1 mm, vias 19 -> 17
- net N$8: track 7.63 -> 23.1 mm, vias 0 -> 2
- net VCC: track 858.1 -> 867.4 mm
- net GND: track 597.6 -> 599.7 mm
- net D8_RX0: track 173.2 -> 171.2 mm
- net D5_: track 107.0 -> 105.3 mm
- net IO_C: track 197.1 -> 195.7 mm
- net D18_: track 3.28 -> 2.68 mm
Other:
- board text added: "snc98 - Slash Number Calculator Rev. 1.2"
- board text removed: "snc98 - Slash Number Calculator Rev. 1.1"
