File: Hardware/eagle/snc98_keyboard_plate.sch (EAGLE design)
At the start: 25 parts

Commit message: V 5.0 Hardware - Design
Other:
- note added: "V 2.0"
- note removed: "1.0"
Changed lines of the file:
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@@
 <text x="149.86" y="30.48" size="3.81" layer="91" ratio="12">snc98 Keyboard Plate </text>
 <text x="149.86" y="25.4" size="2.54" layer="91" ratio="12">by Jens Grabner</text>
-<text x="238.76" y="7.62" size="2.54" layer="91" ratio="12">1.0</text>
+<text x="236.22" y="7.62" size="2.54" layer="91" ratio="12">V 2.0</text>
 <text x="5.08" y="10.16" size="2.1844" layer="91" ratio="10">snc98 3x4 Switch-block Rev. 0.3 by Jens Grabner is licensed under</text>
 <text x="5.08" y="15.24" size="3.81" layer="91" ratio="12">Copyright CERN 2013</text>

Commit message: sinh()_cosh()_tanh() added
Other:
- note added: "V 1.2"
- note removed: "V 2.0"
Changed lines of the file:
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@@
 <text x="149.86" y="30.48" size="3.81" layer="91" ratio="12">snc98 Keyboard Plate </text>
 <text x="149.86" y="25.4" size="2.54" layer="91" ratio="12">by Jens Grabner</text>
-<text x="236.22" y="7.62" size="2.54" layer="91" ratio="12">V 2.0</text>
+<text x="236.22" y="7.62" size="2.54" layer="91" ratio="12">V 1.2</text>
 <text x="5.08" y="10.16" size="2.1844" layer="91" ratio="10">snc98 3x4 Switch-block Rev. 0.3 by Jens Grabner is licensed under</text>
 <text x="5.08" y="15.24" size="3.81" layer="91" ratio="12">Copyright CERN 2013</text>
