File: Hardware/eagle/snc98_3x4_Switch-block.sch (EAGLE design)
At the start: 73 parts

Commit message: cbrt_int96
cbrt added
Parts:
- removed D1, D2, D29, D3, D4, D5: SD103CW, BaseApp:DIODESMA-WIDE
- removed D6, D7, D8: SD103C, BaseApp:DIODE280MIL-TH
- added D01, D02, D03, D04, D05, D06, D07, D08, D09: SD103AW-DIO, BaseApp:DIODESOD-123F
- D10, D11, D12: device BaseApp:DIODESMA-WIDE -> BaseApp:DIODESOD-123F
- D13, D14, D15: value SD103CW -> BAT54A; device BaseApp:DIODESMA-WIDE -> diode:BAT54A; MF MULTICOMP -> (none); MPN SD103CW-7-F -> (none); OC_FARNELL 2306221 -> unknown
- D19, D20, D21: value BAT54A -> SD103C; device diode:BAT54A -> BaseApp:DIODE280MIL-TH; MF (none) -> MULTICOMP; MPN (none) -> SD103CW-7-F; OC_FARNELL unknown -> 2306221
- renumbered D9 to D28
Connections:
- net A_1: now also D01.A, D02.A, D03.A, D04.A, D13.AA, D14.AA, D19.A, D20.A, D21.A; no longer D1.A, D12.A, D13.A, D16.AA, D17.AA, D23.A, D24.A, D27.A, D29.A
- net A_2: now also D05.A, D06.A, D07.A, D08.A, D15.AA, D16.AA, D23.A, D24.A; no longer D11.A, D14.A, D18.AA, D19.AA, D2.A, D25.A, D26.A, D5.A
- net A_3: now also D09.A, D11.A, D12.A, D17.AA, D18.AA, D25.A, D26.A, D27.A; no longer D15.A, D20.AA, D21.AA, D3.A, D4.A, D6.A, D7.A, D8.A
- net N$16: now also D09.C, D17.K1, D25.C; no longer D15.C, D20.K1, D6.C
- net N$18: now also D17.K2, D26.C; no longer D20.K2, D7.C
- net N$19: now also D02.C, D13.K2, D19.C; no longer D12.C, D16.K2, D27.C
- net N$2: now also D04.C, D14.K2, D21.C; no longer D1.C, D17.K2, D23.C
- net N$21: now also D11.C, D18.K1, D27.C; no longer D21.K1, D4.C, D8.C
- net N$22: now also D12.C, D18.K2; no longer D21.K2, D3.C
- net N$24: now also D05.C, D15.K1; no longer D14.C, D18.K1
- net N$25: now also D06.C, D15.K2, D22.C; no longer D11.C, D18.K2, D26.C
- net N$28: now also D07.C, D16.K1, D23.C; no longer D19.K1, D25.C, D5.C
- net N$30: now also D08.C, D16.K2, D24.C; no longer D19.K2, D2.C, D22.C
- net N$32: now also D03.C, D14.K1, D20.C; no longer D17.K1, D24.C, D29.C
- net N$6: now also D01.C, D13.K1; no longer D13.C, D16.K1
Other:
- moved on the sheet: D10, D11, D12, D16, D17, D18, D22, D23, D24, D25, D26, D27

Commit message: add Dokument "The_flipped_continued_fraction.pdf"
Parts:
- removed R2, R3: 6k8, rcl:R-EU_R1206
- removed R23, R25, R27: 27k, rcl:R-EU_0204/5
- removed R24, R26, R28: 6k8, rcl:R-EU_0204/5
- removed R4, R5, R6: 27k, rcl:R-EU_R1206
- removed R7: 6k8, rcl:R-EU_M0805
- removed R9: 27k, rcl:R-EU_M0805
- added R12: 27k, rcl:R-EU_M0805
- R1: device rcl:R-EU_R1206 -> rcl:R-EU_M0805; TME_EU (none) -> RC0805FR-076K8
Connections:
- net A1: now also R12.1; no longer R1.2, R23.1, R24.2, R4.1, R9.1
- net A2: now also R1.2; no longer R2.2, R25.1, R26.2, R5.1, R7.2
- net A3: no longer R27.1, R28.2, R3.2, R6.1
- net AREF: now also R12.2; no longer R23.2, R25.2, R27.2, R4.2, R5.2, R6.2, R9.2
- net A_1: no longer R1.1, R24.1
- net A_2: now also R1.1; no longer R2.1, R26.1, R7.1
- net A_3: no longer R28.1, R3.1
Other:
- note added: "Switches: https://de.aliexpress.com/item/32534955696.html"
- moved on the sheet: R1
