File: Hardware/eagle/snc98_3x4_Switch-cherry_ml.sch (EAGLE design)
At the start: 73 parts

Commit message: add Dokument "The_flipped_continued_fraction.pdf"
Parts:
- added U$1, U$2: CHERRY_MX_2, cherry:CHERRY_MX_2
Changed lines of the file:
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@@
 <setting verticaltext="up"/>
 </settings>
-<grid distance="50" unitdist="mil" unit="mil" style="lines" multiple="1" display="yes" altdistance="0.05" altunitdist="inch" altunit="inch"/>
+<grid distance="0.1" unitdist="inch" unit="inch" style="lines" multiple="1" display="no" altdistance="0.01" altunitdist="inch" altunit="inch"/>
 <layers>
 <layer number="1" name="Top" color="4" fill="1" visible="no" active="no"/>
@@
 <part name="S11" library="ML1A-11JW" deviceset="ML1A-11JW" device=""/>
 <part name="S12" library="ML1A-11JW" deviceset="ML1A-11JW" device=""/>
+<part name="U$1" library="cherry" deviceset="CHERRY_MX_2" device=""/>
+<part name="U$2" library="cherry" deviceset="CHERRY_MX_2" device=""/>
 </parts>
 <sheets>
