File: Hardware/eagle/snc98_3x4_Switch-futuba.sch (EAGLE design)
At the start: 73 parts, among them SW1 CHERRY_MX_WITH_FIXING_PINS, SW10 CHERRY_MX_WITH_FIXING_PINS, SW11 CHERRY_MX_WITH_FIXING_PINS, SW12 CHERRY_MX_WITH_FIXING_PINS, SW2 CHERRY_MX_WITH_FIXING_PINS, SW3 CHERRY_MX_WITH_FIXING_PINS, SW4 CHERRY_MX_WITH_FIXING_PINS, SW5 CHERRY_MX_WITH_FIXING_PINS, SW6 CHERRY_MX_WITH_FIXING_PINS, SW7 CHERRY_MX_WITH_FIXING_PINS, SW8 CHERRY_MX_WITH_FIXING_PINS, SW9 CHERRY_MX_WITH_FIXING_PINS

Commit message: add Dokument "The_flipped_continued_fraction.pdf"
Parts:
- added S1A, S3: CHERRY_MX, cherry:CHERRY_MX
- added SW13: CHERRY_MX_WITH_FIXING_PINS, Cherry_MX_v7.0:CHERRY_MX_WITH_FIXING_PINS
- SW5: value CHERRY_MX_WITH_FIXING_PINS -> CHERRY_MX; device Cherry_MX_v7.0:CHERRY_MX_WITH_FIXING_PINS -> Cherry_MX_v7.0:CHERRY_MX
Connections:
- net C1: now also S1A.1, S3.1, SW13.1
- net N$16: now also S1A.2, S3.2
- net N$6: now also SW13.2
Changed lines of the file:
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@@
 <setting verticaltext="up"/>
 </settings>
-<grid distance="0.1" unitdist="inch" unit="inch" style="lines" multiple="1" display="yes" altdistance="0.05" altunitdist="inch" altunit="inch"/>
+<grid distance="50" unitdist="mil" unit="mil" style="lines" multiple="1" display="no" altdistance="0.01" altunitdist="inch" altunit="inch"/>
 <layers>
 <layer number="1" name="Top" color="4" fill="1" visible="no" active="no"/>
@@
 <part name="SW3" library="Cherry_MX_v7.0" deviceset="CHERRY_MX" device="_WITH_FIXING_PINS"/>
 <part name="SW4" library="Cherry_MX_v7.0" deviceset="CHERRY_MX" device="_WITH_FIXING_PINS"/>
-<part name="SW5" library="Cherry_MX_v7.0" deviceset="CHERRY_MX" device="_WITH_FIXING_PINS"/>
+<part name="SW5" library="Cherry_MX_v7.0" deviceset="CHERRY_MX" device="" value="CHERRY_MX"/>
 <part name="SW6" library="Cherry_MX_v7.0" deviceset="CHERRY_MX" device="_WITH_FIXING_PINS"/>
 <part name="SW7" library="Cherry_MX_v7.0" deviceset="CHERRY_MX" device="_WITH_FIXING_PINS"/>
@@
 <part name="SW11" library="Cherry_MX_v7.0" deviceset="CHERRY_MX" device="_WITH_FIXING_PINS"/>
 <part name="SW12" library="Cherry_MX_v7.0" deviceset="CHERRY_MX" device="_WITH_FIXING_PINS"/>
+<part name="SW13" library="Cherry_MX_v7.0" deviceset="CHERRY_MX" device="_WITH_FIXING_PINS"/>
+<part name="S1A" library="cherry" deviceset="CHERRY_MX" device=""/>
+<part name="S3" library="cherry" deviceset="CHERRY_MX" device=""/>
 </parts>
 <sheets>
@@
 <instance part="SW11" gate="G$1" x="220.98" y="93.98" rot="R90"/>
 <instance part="SW12" gate="G$1" x="220.98" y="66.04" rot="R90"/>
+<instance part="SW13" gate="G$1" x="137.16" y="137.16" rot="R90"/>
+<instance part="S1A" gate="G$1" x="220.98" y="152.4"/>
+<instance part="S3" gate="G$1" x="222.25" y="161.29"/>
 </instances>
 <busses>
@@
 <junction x="151.13" y="149.86"/>
 <wire x1="151.13" y1="147.32" x2="151.13" y2="144.78" width="0.1524" layer="91"/>
-<wire x1="151.13" y1="144.78" x2="182.88" y2="144.78" width="0.1524" layer="91"/>
+<wire x1="151.13" y1="144.78" x2="154.94" y2="144.78" width="0.1524" layer="91"/>
+<wire x1="154.94" y1="144.78" x2="182.88" y2="144.78" width="0.1524" layer="91"/>
 <wire x1="184.15" y1="152.4" x2="182.88" y2="152.4" width="0.1524" layer="91"/>
 <wire x1="182.88" y1="152.4" x2="182.88" y2="149.86" width="0.1524" layer="91"/>
@@
 <wire x1="215.9" y1="147.32" x2="214.63" y2="147.32" width="0.1524" layer="91"/>
 <junction x="214.63" y="147.32"/>
+<pinref part="SW13" gate="G$1" pin="1"/>
+<wire x1="132.08" y1="132.08" x2="154.94" y2="132.08" width="0.1524" layer="91"/>
+<wire x1="154.94" y1="132.08" x2="154.94" y2="144.78" width="0.1524" layer="91"/>
+<junction x="154.94" y="144.78"/>
+<pinref part="S1A" gate="G$1" pin="1"/>
+<pinref part="S3" gate="G$1" pin="1"/>
+<wire x1="217.17" y1="161.29" x2="214.63" y2="161.29" width="0.1524" layer="91"/>
+<wire x1="214.63" y1="161.29" x2="214.63" y2="152.4" width="0.1524" layer="91"/>
+<junction x="214.63" y="152.4"/>
 </segment>
 <segment>
@@
 <pinref part="D25" gate="G$1" pin="C"/>
 <wire x1="232.41" y1="165.1" x2="227.33" y2="165.1" width="0.1524" layer="91"/>
-<wire x1="227.33" y1="165.1" x2="227.33" y2="157.48" width="0.1524" layer="91"/>
+<wire x1="227.33" y1="165.1" x2="227.33" y2="161.29" width="0.1524" layer="91"/>
 <pinref part="D09" gate="G$1" pin="C"/>
+<wire x1="227.33" y1="161.29" x2="227.33" y2="157.48" width="0.1524" layer="91"/>
 <wire x1="227.33" y1="157.48" x2="227.33" y2="154.94" width="0.1524" layer="91"/>
 <wire x1="227.33" y1="154.94" x2="227.33" y2="152.4" width="0.1524" layer="91"/>
@@
 <wire x1="226.06" y1="157.48" x2="227.33" y2="157.48" width="0.1524" layer="91"/>
 <junction x="227.33" y="157.48"/>
+<pinref part="S1A" gate="G$1" pin="2"/>
+<pinref part="S3" gate="G$1" pin="2"/>
+<junction x="227.33" y="161.29"/>
 </segment>
 </net>
@@
 <wire x1="162.56" y1="149.86" x2="163.83" y2="149.86" width="0.1524" layer="91"/>
 <wire x1="163.83" y1="149.86" x2="163.83" y2="152.4" width="0.1524" layer="91"/>
-<wire x1="163.83" y1="152.4" x2="162.56" y2="152.4" width="0.1524" layer="91"/>
 <junction x="163.83" y="152.4"/>
 <pinref part="D13" gate="G$1" pin="K1"/>
@@
 <wire x1="162.56" y1="157.48" x2="163.83" y2="157.48" width="0.1524" layer="91"/>
 <junction x="163.83" y="157.48"/>
-</segment>
-</net>
+<pinref part="SW13" gate="G$1" pin="2"/>
+<wire x1="142.24" y1="142.24" x2="160.02" y2="142.24" width="0.1524" layer="91"/>
+<wire x1="160.02" y1="142.24" x2="160.02" y2="152.4" width="0.1524" layer="91"/>
+<wire x1="160.02" y1="152.4" x2="163.83" y2="152.4" width="0.1524" layer="91"/>
+<label x="160.02" y="142.24" size="1.778" layer="95" rot="R270"/>
+</segment>
+</net>
